Commit message: 민재야 백파일 로깅 가져가라

File: test_pkg/models/model.urdf (robot description, URDF)
Before this commit: robot manipulator, 5 links, 4 joints
Links:
- removed link cf2
- removed link curvature_link
- removed link sphere_link
- added link box_link; visual box size=0.01 2 1
- added link cf2_visual, mass 1; visual mesh filename=package://test_pkg/models/meshes/crazyflie.dae scale=0.001 0.001 0.001
Joints:
- removed joint world_to_curvature
- removed joint world_to_sphere
- added joint world_to_box: type fixed, parent world, child box_link, origin xyz=1.18 0 1.5 rpy=0 0 0
- joint drone_to_ee: parent cf2 -> cf2_visual
- joint world_to_drone: child cf2 -> cf2_visual

Commit message: 2022 법벡추 kroc버전으로 리턴

File: test_pkg/models/model.urdf (robot description, URDF)
Before this commit: robot manipulator, 4 links, 3 joints
Links:
- removed link box_link
- added link curvature; visual mesh filename=package://test_pkg/models/meshes/curvature.dae scale=0.01 0.02 0.02
Joints:
- removed joint world_to_box
- added joint world_to_curvature: type fixed, parent world, child curvature, origin xyz=0.5 3.8 0 rpy=0 0 0
